File: DiscTransmitter.sch (KiCad schematic (older format))
At the start: 41 parts, among them J1 Conn_01x01_Male, J2 Conn_01x01_Male, J3 Conn_01x04_Male, J4 Conn_01x01_Male, U1 SNx4HC595_8b_Shift_Reg, U2 4-DigitSevenSegment, U3 SNx4HC595_8b_Shift_Reg, U4 SNx4HC595_8b_Shift_Reg, U5 SNx4HC595_8b_Shift_Reg

Commit message: Fixed pads on RFM footprint
Parts:
- J1, J2, J4: symbol conn:Conn_01x01_Male -> DiscTransmitter-rescue:Conn_01x01_Male-conn
- J3: symbol conn:Conn_01x04_Male -> DiscTransmitter-rescue:Conn_01x04_Male-conn
- U2: footprint my_foot_prints:FourDigitSevenSegmentDisplay -> my_foot_prints:TwoDigDisplayX2
Changed lines of the file:
@@
 F 0 "U2" H 7350 3200 60  0000 C CNN
 F 1 "4-DigitSevenSegment" H 7800 3950 39  0000 C CNN
-F 2 "my_foot_prints:FourDigitSevenSegmentDisplay" H 7350 3200 60  0001 C CNN
+F 2 "my_foot_prints:TwoDigDisplayX2" H 7350 3200 60  0001 C CNN
 F 3 "" H 7350 3200 60  0001 C CNN
 	1    7350 3400
@@
 Connection ~ 4700 6500
 $Comp
-L conn:Conn_01x04_Male J3
+L DiscTransmitter-rescue:Conn_01x04_Male-conn J3
 U 1 1 5B3577AF
 P 4300 7600
@@
 $EndComp
 $Comp
-L conn:Conn_01x01_Male J4
+L DiscTransmitter-rescue:Conn_01x01_Male-conn J4
 U 1 1 5B35782A
 P 5000 7400
@@
 $EndComp
 $Comp
-L conn:Conn_01x01_Male J2
+L DiscTransmitter-rescue:Conn_01x01_Male-conn J2
 U 1 1 5B3578C4
 P 3900 7650
@@
 $EndComp
 $Comp
-L conn:Conn_01x01_Male J1
+L DiscTransmitter-rescue:Conn_01x01_Male-conn J1
 U 1 1 5B357982
 P 3750 7500
