File: Transmitter board/Transmitter board.sch (KiCad schematic (older format))
At the start: 25 parts, among them J3 Conn_01x02_Male, J4 Conn_01x03_Male, J5 Conn_01x04_Male, J6 Conn_01x03_Male, J7 Conn_01x05_Male, J8 Conn_01x02_Male, SW1 SW_Push, U1 RFM69HCW, U2 LPC824_HVQFN33, U3 SWD_10-pin-1.27_Conn_2x5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

Commit message: new commit.
Parts:
- R8: value 750ohm -> 330ohm
Changed lines of the file:
@@
 P 10500 5300
 F 0 "R8" H 10600 5350 50  0000 L CNN
-F 1 "750ohm" H 10600 5250 50  0000 L CNN
+F 1 "330ohm" H 10600 5250 50  0000 L CNN
 F 2 "my_foot_prints:R_0402" H 10500 5300 50  0001 C CNN
 F 3 "~" H 10500 5300 50  0001 C CNN

Commit message: Fixed pads on RFM footprint
Parts:
- U1: footprint my_foot_prints:RFM96C -> my_foot_prints:RFM96HCW
Changed lines of the file:
@@
 EESchema Schematic File Version 4
+LIBS:Transmitter board-cache
 EELAYER 26 0
 EELAYER END
@@
 F 0 "U1" H 2650 6450 60  0000 C CNN
 F 1 "RFM69HCW" V 2650 6100 60  0000 C CNN
-F 2 "my_foot_prints:RFM96C" H 2650 6100 60  0001 C CNN
+F 2 "my_foot_prints:RFM96HCW" H 2650 6100 60  0001 C CNN
 F 3 "" H 2650 6100 60  0001 C CNN
 	1    2650 6100
