File: Minimized Transmitter/Minimized Transmitter.sch (KiCad schematic (older format))
At the start: 8 parts, among them J1 Conn_ARM_JTAG_SWD_10, J2 Conn_01x02_Male, J3 Conn_01x03_Male, U1 LPC824M201JHI33, U2 RFM69HCW

Commit message: test
Parts:
- U2: symbol Transmitter~board-rescue:RFM69HCW -> Minimized-Transmitter-rescue:RFM69HCW-Transmitter~board-rescue
Changed lines of the file:
@@
 $EndComp
 $Comp
-L Transmitter~board-rescue:RFM69HCW U2
+L Minimized-Transmitter-rescue:RFM69HCW-Transmitter~board-rescue U2
 U 1 1 5C15B19A
 P 6900 4500
